File: basement_humidity/basement_humidity.kicad_pcb (KiCad board)
At the start: 2 copper layers, 9 parts, among them J1 Screw_Terminal_01x02, J2 Screw_Terminal_01x03, U1 NRF24L01_Breakout, U2 DHT11

Commit message: initial
Parts:
- C2: footprint Capacitor_THT:C_Disc_D5.0mm_W2.5mm_P2.50mm -> Capacitor_THT:C_Disc_D5.0mm_W2.5mm_P5.00mm
- R1: footprint Resistor_THT:R_Axial_DIN0207_L6.3mm_D2.5mm_P15.24mm_Horizontal -> Resistor_THT:R_Axial_DIN0411_L9.9mm_D3.6mm_P7.62mm_Vertical
- moved C2 78.9 mm to (176.5, 100.3)
- moved U1 73.9 mm to (168.9, 105.4), turned to 0 degrees
- moved R1 48.3 mm to (138.4, 82.5), turned to 90 degrees
- moved D1 47.3 mm to (138.4, 90.2)
- moved J2 43.2 mm to (181.6, 69.8)
- moved U2 43.0 mm to (180.3, 86.4)
- moved A1 35.9 mm to (146.1, 72.4)
- moved C1 35.9 mm to (148.6, 62.2)
- moved J1 35.9 mm to (151.1, 50.8)
Connections:
- A1 pad 29: Net-(A1-Pad29) -> GND
- U1 pad 3: Net-(A1-Pad15) -> Net-(A1-Pad12)
- U2 pad 2: Net-(U2-Pad2) -> Net-(A1-Pad19)
- U2 pad 4: Net-(U2-Pad4) -> GND
Routing:
- net Net-(A1-Pad15): track 80.1 -> 0.00 mm
- net +5V: track 160.1 -> 120.2 mm
- net Net-(A1-Pad10): track 36.1 -> 69.5 mm
- net Net-(A1-Pad11): track 31.2 -> 59.4 mm
- net Net-(A1-Pad12): track 0.00 -> 28.1 mm
- net Net-(A1-Pad14): track 48.5 -> 27.1 mm
- net Net-(A1-Pad20): track 25.1 -> 45.2 mm
- net GND: track 167.7 -> 148.8 mm
- net Net-(A1-Pad13): track 46.7 -> 29.3 mm
- net Net-(D1-Pad1): track 0.00 -> 7.62 mm
- net Net-(A1-Pad19): track 20.1 -> 27.4 mm
- net Net-(A1-Pad8): track 0.00 -> 5.08 mm
Other:
- rule via_min_size: 0.4 -> 0.2
