File: basement_humidity/basement_humidity.sch (KiCad schematic (older format))
At the start: 9 parts, among them J1 Screw_Terminal_01x02, J2 Screw_Terminal_01x03, U1 NRF24L01_Breakout, U2 DHT11

Commit message: initial
Changed lines of the file:
@@
 	5050 4550 2500 4550
-Wire Wire Line
-	6600 2800 6600 4850
-Wire Wire Line
-	6600 4850 1900 4850
 Wire Wire Line
 	7250 700  7250 750
@@
 $EndComp
 $Comp
-L power:+5V #PWR0107
-U 1 1 5D29D7E7
-P 3800 1900
-F 0 "#PWR0107" H 3800 1750 50  0001 C CNN
-F 1 "+5V" H 3815 2073 50  0000 C CNN
-F 2 "" H 3800 1900 50  0001 C CNN
-F 3 "" H 3800 1900 50  0001 C CNN
-	1    3800 1900
-	1    0    0    -1
-$EndComp
-$Comp
 L Connector:Screw_Terminal_01x02 J1
 U 1 1 5D29E49A
@@
 Wire Wire Line
 	7250 2800 7400 2800
-Wire Wire Line
-	6600 2800 7250 2800
-Connection ~ 7250 2800
 $Comp
 L RF:NRF24L01_Breakout U1
@@
 	4700 1200 4700 3000
 Wire Wire Line
-	1900 3500 3100 3500
-Wire Wire Line
-	1900 3500 1900 4850
-Wire Wire Line
 	3100 3100 2400 3100
 Wire Wire Line
@@
 	1    0    0    -1
 $EndComp
+Wire Wire Line
+	3100 3200 1750 3200
+Wire Wire Line
+	1750 3200 1750 5250
+Wire Wire Line
+	1750 5250 7050 5250
+Wire Wire Line
+	7050 5250 7050 2800
+Wire Wire Line
+	7050 2800 7250 2800
+Connection ~ 7250 2800
+$Comp
+L power:GND #PWR?
+U 1 1 5D2BFDAA
+P 5350 2200
+F 0 "#PWR?" H 5350 1950 50  0001 C CNN
+F 1 "GND" H 5355 2027 50  0000 C CNN
+F 2 "" H 5350 2200 50  0001 C CNN
+F 3 "" H 5350 2200 50  0001 C CNN
+	1    5350 2200
+	1    0    0    -1
+$EndComp
